File: electronics/kicad/Faceboard/Faceboard.kicad_pcb (KiCad board)
At the start: 2 copper layers, 48.7 x 48.9 mm, 17 parts, among them J10 Gnd, J11 Primary Trigger 1, J12 Secondary Trigger, J13 Head Button, J14 Base Button, J15 Conn_01x05, J16 Conn_01x05, J17 Conn_01x05, J18 Conn_01x05, M2.5 MountingHole_2.7mm_M2.5_DIN96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, U4 Face Hat Top, U5 Face Hat Right, U6 Face Hat Left, U7 Face Button

Commit message: Updated Schematic
Some Parts were replaced with Hand Solder SMD components where possible. Routing changed to work with new parts
Parts:
- removed G***: LOGO, Custom Footprint Library:yoi-con
