File: electronics/kicad/Mainboard/Mainboard.kicad_pcb (KiCad board)
At the start: 2 copper layers, 99 x 53 mm, 30 parts, among them J1 GND Pair, J10 Conn_01x05, J11 Box Switch 1, J12 Box Switch 2, J13 Bos Switch 3, J14 LED Strip, J2 X-Axis Hall, J3 Y-Axis Hall, J4 Conn_01x05, J5 Conn_01x05, J6 USB_A_Stacked, J7 Conn_01x05, J8 Conn_01x05, J9 Conn_01x05, M2.5 MountingHole_2.7mm_M2.5_DIN96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, U1 ESP32-C6-DevKitC-1, U3 MCP23017x-x-SO

Commit message: -
Parts:
- R1, R2: value 2.2K -> 2K2
