File: electronics/kicad/Mainboard/Mainboard.kicad_sch (KiCad schematic)
At the start: 19 parts, among them J1 GND Pair, J10 Conn_01x05, J11 Box Switch 1, J12 Box Switch 2, J13 Bos Switch 3, J14 LED Strip, J2 X-Axis Hall, J3 Y-Axis Hall, J4 Conn_01x05, J5 Conn_01x05, J6 USB_A_Stacked, J7 Conn_01x05, J8 Conn_01x05, J9 Conn_01x05, U1 ESP32-C6-DevKitC-1, U2 MCP23017_SP

Commit message: Updated Schematic
Some Parts were replaced with Hand Solder SMD components where possible. Routing changed to work with new parts
Parts:
- removed U2: MCP23017_SP, Package_DIP:DIP-28_W7.62mm, symbol Interface_Expansion:MCP23017_SP
- added U3: MCP23017x-x-SO, Package_SO:SOIC-28W_7.5x17.9mm_P1.27mm, symbol Interface_Expansion:MCP23017x-x-SO
- J6: footprint Connector_USB:USB_A_CUI_UJ2-ADH-TH_Horizontal_Stacked -> Connector_USB:USB_A_Wuerth_61400826021_Horizontal_Stacked
- R1, R2, R3: footprint Resistor_THT:R_Axial_DIN0204_L3.6mm_D1.6mm_P5.08mm_Horizontal -> Resistor_SMD:R_1206_3216Metric_Pad1.30x1.75mm_HandSolder
Connections:
- net Base Button: now also J5.1 (Pin_1); no longer J5.3 (Pin_3)
- net Face Button: now also J5.3 (Pin_3); no longer J5.5 (Pin_5)
- net Face Hat Left - Center: now also U3.21 (GPA0)
- net Face Hat Left - Down: now also U3.23 (GPA2)
- net Face Hat Left - Left: now also U3.22 (GPA1)
- net Face Hat Left - Right: now also U3.24 (GPA3)
- net Face Hat Left - Up: now also U3.25 (GPA4)
- net Face Hat Right - Center: now also J8.3 (Pin_3), U3.1 (GPB0); no longer J8.1 (Pin_1)
- net Face Hat Right - Down: now also J8.1 (Pin_1); no longer J8.3 (Pin_3)
- net Face Hat Right - Left: now also U3.2 (GPB1)
- net Face Hat Right - Right: now also U3.27 (GPA6)
- net Face Hat Right - Up: now also U3.26 (GPA5)
- net GND: now also U3.10 (V_{SS}), U3.15 (A0), U3.16 (A1), U3.17 (A2)
- net Head Button: now also J5.2 (Pin_2); no longer J5.4 (Pin_4)
- net INT: now also U3.19 (INTB), U3.20 (INTA)
- net Primary Trigger: now also J5.5 (Pin_5); no longer J5.1 (Pin_1)
- net SCK: now also U1.5 (GPIO6), U3.12 (SCK); no longer U1.6 (GPIO7)
- net SDA: now also U1.6 (GPIO7), U3.13 (SDA); no longer U1.5 (GPIO6)
- net Secondary Trigger: now also J5.4 (Pin_4); no longer J5.2 (Pin_2)
- net Thumb Hat - Center: now also U3.6 (GPB5)
- net Thumb Hat - Down: now also U3.3 (GPB2)
- net Thumb Hat - Left: now also U3.7 (GPB6)
- net Thumb Hat - Right: now also U3.4 (GPB3)
- net Thumb Hat - Up: now also U3.5 (GPB4)
- net Vcc renamed 3V3
- net 3V3: now also U3.18 (~{RESET}), U3.9 (V_{DD})
Other:
- moved on the sheet: R1, R2

Commit message: -
Parts:
- R1, R2: value 2.2K -> 2K2
Changed lines of the file:
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@@
 			)
 		)
-		(property "Value" "2.2K"
+		(property "Value" "2K2"
 			(at 201.93 44.4499 0)
 			(show_name no)
@@
 			)
 		)
-		(property "Value" "2.2K"
+		(property "Value" "2K2"
 			(at 210.82 44.4499 0)
 			(show_name no)
